File: Fume Extractor/board.brd (EAGLE design)
At the start: 40 x 60 mm, 26 parts, among them IC1 DW01, IC2 BQ21040DBVR, J1 TYPE-C-31-M-17, T1 FS8205A, U1 MT3608

Commit message: PCB layout update
Parts:
- added C9: 22uF, rcl:C0805
- added JP3: (no value), pinhead_v2:1X02/OCT
- C1: value 0.1uF -> 1uF; device rcl:C0805 -> rcl:C0603
- C2: value 4.7uF -> 1uF; device rcl:C0805 -> rcl:C0603
- C3: value 4.7uF -> 1uF
- C4: value 22uF -> 100nF; device rcl:C0805 -> rcl:C0603
- C5: value 4.7uF -> 100nF; device rcl:C0805 -> rcl:C0603
- C7: value 10uF -> 4.7uF; device rcl:SMC_A -> rcl:C0603
- C8: value 4.7uF -> 10uF; device rcl:C0603 -> rcl:C0805
- IC1: value DW01 -> BQ21040DBVR; device DW01:SOT95P280X135-6N -> SamacSys_Parts:SOT95P280X145-6N
- IC2: value BQ21040DBVR -> DW01; device SamacSys_Parts:SOT95P280X145-6N -> DW01:SOT95P280X135-6N
- LED1: device led:CHIP-LED0603 -> led:CHIP-LED0805
- R1: value 100 -> 1k; device rcl:R0805 -> rcl:R0603
- R2: value 1k -> 1.5k; device rcl:R0805 -> rcl:R0603
- R3: device rcl:R0402 -> rcl:R0603
- R4: value 8.2k -> 100Ω; device rcl:R0805 -> rcl:R0603
- R5: value 430Ω -> 1k; device rcl:R0805 -> rcl:R0603
- R6: value 10k -> 8.2k; device rcl:R0402 -> rcl:R0603
- R7: value 1.5k -> 430Ω; device rcl:R0402 -> rcl:R0603
- moved R4 67.6 mm to (35.1, 8.38), turned to 90 degrees
- moved C1 64.7 mm to (20.1, 9.14)
- moved D1 64.3 mm to (21.1, 11.4)
- moved C4 59.5 mm to (31.6, 5.33), turned to 180 degrees
- moved T1 58.8 mm to (31.5, 12.7), turned to 90 degrees
- moved IC2 58.8 mm to (31.8, 8.38)
- moved R3 58.4 mm to (7.87, 9.65), turned to 180 degrees
- moved J1 55.6 mm to (20.1, 6.35)
- moved R5 54.5 mm to (28.4, 8.38), turned to 270 degrees
- moved R6 51.7 mm to (11.4, 25.9), turned to 180 degrees
- moved R2 51.6 mm to (4.83, 2.54), turned to 180 degrees
- moved LED1 50.7 mm to (2.54, 6.10), turned to 180 degrees
- moved U1 50.0 mm to (11.2, 22.6), turned to 180 degrees
- moved R1 49.9 mm to (7.87, 2.54), turned to 180 degrees
- moved R7 49.7 mm to (14.5, 25.9), turned to 180 degrees
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Connections:
- net 12V: now also C7.1, C8.1, C9.1, R6.2; no longer C5.1, C6.1, C7.+, R4.1
- net 5V: now also C2.1, C5.1, C6.1, IC1.6; no longer C3.1, C4.1, IC2.6
- net BATT_GND: now also C4.2, IC2.6, JP3.2; no longer C1.2, IC1.6
- net GND: now also C1.2, C7.2, C9.2, IC1.5, R1.1, R3.1, R7.1; no longer C4.2, C7.-, IC2.5, R2.1, R3.2, R6.1
- net N$1: now also IC2.5, R4.2; no longer IC1.5, R1.2
- net N$12: now also R6.1, R7.2; no longer R4.2, R5.1
- net N$13: now also C1.1; no longer C2.1
- net N$2: now also IC1.1, R3.2; no longer IC2.1, R6.2
- net N$3: now also IC1.3, R2.1; no longer IC2.3, R7.2
- net N$4: now also IC2.2, R5.1; no longer IC1.2, R2.2
- net N$6: now also IC2.1; no longer IC1.1
- net N$7: now also IC2.3; no longer IC1.3
- net N$8: now also R2.2; no longer R7.1
- net N$9: now also IC1.4, R1.2; no longer IC2.4, R3.1
- net V_BATT: now also C3.1, C4.1, IC1.2, JP3.1, R4.1; no longer C1.1, C8.1, IC2.2, R1.1
Routing:
- added copper zone on layer 1, net GND
- added copper zone on layer 16, net GND
Other:
- board size 40 x 60 mm -> 40 x 40 mm
- board text added: "+"
- board text added: "-"
- board text added: "BATT"

Commit message: PCB layout update;
Parts:
- added C10, C11: 100nF, rcl:C0603
- added C12: 3nF, rcl:C0603
- added D3, D4: SS34, diode:DO214AC
- added IC3: TLC555, linear:SO08
- added J2: (no value), SparkFun-Connectors:MOLEX-1X4_LOCK
- moved C9 12.9 mm to (14.7, 17.3), turned to 0 degrees
- moved C8 11.8 mm to (14.7, 19.3), turned to 0 degrees
- moved C7 10.8 mm to (14.2, 21.3), turned to 0 degrees
- moved R7 9.66 mm to (10.2, 17.3), turned to 90 degrees
- moved C6 9.43 mm to (2.29, 16.8), turned to 270 degrees
- moved R6 8.64 mm to (11.7, 17.3), turned to 90 degrees
- moved C5 8.44 mm to (4.32, 16.5), turned to 270 degrees
- moved U1 6.55 mm to (7.37, 17.3), turned to 90 degrees
- moved D2 6.51 mm to (11.2, 22.4), turned to 90 degrees
- moved JP3 3.84 mm to (33.0, 2.79), turned to 180 degrees
- moved L1 2.09 mm to (5.33, 22.6), turned to 0 degrees
- moved T1 1.55 mm to (33.0, 13.0)
- moved IC2 1.55 mm to (33.3, 8.64)
- moved R4 1.55 mm to (36.6, 8.64)
- moved R5 1.55 mm to (30.0, 8.64), turned to 90 degrees
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Connections:
- new net N$11: C10.1, IC3.5
- new net N$15: C12.1, D3.A, D4.C, IC3.2, IC3.6
- new net N$16: D3.C
- new net N$17: D4.A
- new net PWM: IC3.3
- net 12V: now also C11.2, IC3.4, IC3.8, J2.2
- net GND: now also C10.2, C11.1, C12.2, IC3.1, J2.1
Routing:
- net V_BATT: track 0.00 -> 14.4 mm
- net BATT_GND: track 0.00 -> 13.3 mm
- net N$7: track 0.00 -> 12.5 mm
- net N$14: track 0.00 -> 11.8 mm
- net N$5: track 0.00 -> 10.6 mm
- net N$6: track 0.00 -> 6.37 mm
- net N$3: track 0.00 -> 5.48 mm
- net N$9: track 0.00 -> 3.72 mm
- net N$8: track 0.00 -> 3.14 mm
- net N$4: track 0.00 -> 2.70 mm
- net N$1: track 0.00 -> 2.55 mm
- net N$2: track 0.00 -> 2.52 mm
- net 5V: track 0.00 -> 2.50 mm
- net N$13: track 0.00 -> 2.36 mm
Other:
- outline, holes or cut-outs redrawn
- board text added: "12V"
- board text added: "GND"
- board text added: "PWM"
- board text added: "TACH"
