File: Fume Extractor/board.sch (EAGLE design)
At the start: 26 parts, among them IC1 BQ21040DBVR, IC2 DW01, J1 TYPE-C-31-M-17, T1 FS8205A, U2 MT3608

Commit message: added PCB design
Parts:
- removed C13: 4.7uF, rcl:C-EUC0603
- removed C9: 0.1uF, rcl:C-EUC0805
- removed JP3: JUMPER-SMT_2_NO_NO-SILK, SparkFun-Jumpers:JUMPER-SMT_2_NO_NO-SILK
- added C2: 4.7uF, rcl:C-EUC0805
- added C4: 22uF, rcl:C-EUC0805
- added JP2: current, pinhead_v2:PINHD-1X2/OCT
- C1: value 4.7uF -> 0.1uF
- C8: value 22uF -> 4.7uF; device rcl:C-EUC0805 -> rcl:C-EUC0603
- IC1: value BQ21040DBVR -> DW01; device SamacSys_Parts:BQ21040DBVR -> DW01:DW01
- IC2: value DW01 -> BQ21040DBVR; device DW01:DW01 -> SamacSys_Parts:BQ21040DBVR
- JP1: value current -> JUMPER-SMT_2_NO_NO-SILK; device pinhead_v2:PINHD-1X2/OCT -> SparkFun-Jumpers:JUMPER-SMT_2_NO_NO-SILK
- R1: value 10k -> 100; device rcl:R-US_R0402 -> rcl:R-US_R0805
- R2: value 10k -> 1k; device rcl:R-US_R0402 -> rcl:R-US_R0805
- R3: value 1.5k -> 10k
- R5: value 100 -> 430Ω
- R6: value 1k -> 10k; device rcl:R-US_R0805 -> rcl:R-US_R0402
- R7: value 430Ω -> 1.5k; device rcl:R-US_R0805 -> rcl:R-US_R0402
- renumbered C14 to C3, U2 to U1
Connections:
- net 5V: now also C4.1, IC2.VIN, JP1.2, JP2.1; no longer C8.1, IC1.VIN, JP1.1, JP3.2
- net BATT_GND: now also C1.2, IC1.VSS; no longer C9.2, IC2.VSS
- net GND: now also C2.2, C4.2, IC2.GND, R2.1, R3.2, R5.2; no longer C1.2, C13.2, IC1.GND, R1.1, R2.2, R7.2
- net N$1: now also IC1.VDD, R1.2; no longer IC2.VDD, R5.2
- net N$12: now also R5.1; no longer R7.1
- net N$13: now also C2.1, JP1.1, JP2.2; no longer C1.1, JP1.2, JP3.1
- net N$2: now also IC2.TS, R6.2; no longer IC1.TS, R1.2
- net N$3: now also IC2.!CHG, R7.2; no longer IC1.!CHG, R3.2
- net N$4: now also IC1.CSI, R2.2; no longer IC2.CSI, R6.2
- net N$6: now also IC1.OD; no longer IC2.OD
- net N$7: now also IC1.OC; no longer IC2.OC
- net N$8: now also R7.1; no longer R3.1
- net N$9: now also IC2.ISET, R3.1; no longer IC1.ISET, R2.1
- net V_BATT: now also C1.1, C8.1, IC2.OUT, R1.1; no longer C13.1, C9.1, IC1.OUT, R5.1
Other:
- moved on the sheet: C1, C5, C6, C7, C8, D2, L1, R1, R2, R3, R4, R5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

Commit message: PCB layout update
Parts:
- added C9: 22uF, rcl:C-EUC0805
- added JP3: (no value), pinhead_v2:PINHD-1X2/OCT
- C1: value 0.1uF -> 1uF; device rcl:C-EUC0805 -> rcl:C-EUC0603
- C2: value 4.7uF -> 1uF; device rcl:C-EUC0805 -> rcl:C-EUC0603
- C3: value 4.7uF -> 1uF
- C4: value 22uF -> 100nF; device rcl:C-EUC0805 -> rcl:C-EUC0603
- C5: value 4.7uF -> 100nF; device rcl:C-EUC0805 -> rcl:C-EUC0603
- C7: value 10uF -> 4.7uF; device rcl:CPOL-USSMCA -> rcl:C-EUC0603
- C8: value 4.7uF -> 10uF; device rcl:C-EUC0603 -> rcl:C-EUC0805
- IC1: value DW01 -> BQ21040DBVR; device DW01:DW01 -> SamacSys_Parts:BQ21040DBVR
- IC2: value BQ21040DBVR -> DW01; device SamacSys_Parts:BQ21040DBVR -> DW01:DW01
- LED1: device led:LEDCHIP-LED0603 -> led:LEDCHIP-LED0805
- R1: value 100 -> 1k; device rcl:R-US_R0805 -> rcl:R-US_R0603
- R2: value 1k -> 1.5k; device rcl:R-US_R0805 -> rcl:R-US_R0603
- R3: device rcl:R-US_R0402 -> rcl:R-US_R0603
- R4: value 8.2k -> 100Ω; device rcl:R-US_R0805 -> rcl:R-US_R0603
- R5: value 430Ω -> 1k; device rcl:R-US_R0805 -> rcl:R-US_R0603
- R6: value 10k -> 8.2k; device rcl:R-US_R0402 -> rcl:R-US_R0603
- R7: value 1.5k -> 430Ω; device rcl:R-US_R0402 -> rcl:R-US_R0603
Connections:
- net 12V: now also C7.1, C8.1, C9.1, R6.2; no longer C5.1, C6.1, C7.+, R4.1
- net 5V: now also C2.1, C5.1, C6.1, IC1.VIN; no longer C3.1, C4.1, IC2.VIN
- net BATT_GND: now also C4.2, IC2.VSS, JP3.2; no longer C1.2, IC1.VSS
- net GND: now also C1.2, C7.2, C9.2, IC1.GND, R1.1, R3.1, R7.1; no longer C4.2, C7.-, IC2.GND, R2.1, R3.2, R6.1
- net N$1: now also IC2.VDD, R4.2; no longer IC1.VDD, R1.2
- net N$12: now also R6.1, R7.2; no longer R4.2, R5.1
- net N$13: now also C1.1; no longer C2.1
- net N$2: now also IC1.TS, R3.2; no longer IC2.TS, R6.2
- net N$3: now also IC1.!CHG, R2.1; no longer IC2.!CHG, R7.2
- net N$4: now also IC2.CSI, R5.1; no longer IC1.CSI, R2.2
- net N$6: now also IC2.OD; no longer IC1.OD
- net N$7: now also IC2.OC; no longer IC1.OC
- net N$8: now also R2.2; no longer R7.1
- net N$9: now also IC1.ISET, R1.2; no longer IC2.ISET, R3.1
- net V_BATT: now also C3.1, C4.1, IC1.OUT, JP3.1, R4.1; no longer C1.1, C8.1, IC2.OUT, R1.1
Other:
- moved on the sheet: C1, C2, C3, C4, D1, J1, JP1, JP2, R1, R2, R3, R4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

Commit message: PCB layout update;
Parts:
- added C10, C11: 100nF, rcl:C-EUC0603
- added C12: 3nF, rcl:C-EUC0603
- added D3, D4: SS34, diode:DIODE-DO214AC
- added IC3: TLC555, linear:NE555D
- added J2: (no value), SparkFun-Connectors:CONN_04POLAR_LOCK
Connections:
- new net N$11: C10.1, IC3.CV
- new net N$15: C12.1, D3.A, D4.C, IC3.THR, IC3.TR
- new net N$16: D3.C
- new net N$17: D4.A
- new net PWM: IC3.Q
- net 12V: now also C11.2, IC3.R, IC3.V+, J2.2
- net GND: now also C10.2, C11.1, C12.2, IC3.GND, J2.1
Other:
- moved on the sheet: JP3
